File: Sunrise clock display board/Sunrise clock display board.kicad_pcb (KiCad board)
At the start: 2 copper layers, 160 x 45.7 mm, 20 parts, among them J1 Conn_02x05_Odd_Even, Q1 2N7002, U1 Nokia_5110_display, U2 Nokia_5110_display, U3 Nokia_5110_display

Commit message: Now in stereo if you want.
Parts:
- added LOGO1: Logo_Open_Hardware_Large, Symbol:OSHW-Logo_19x20mm_SilkScreen, B.Cu at (151.1, 101.6)
Other:
- board text added: "Sunrise clock display board V1.0, 2021-04-10 https://github.com/atoomnetmarc/Sunrise-clock-hardware Apache License, Version 2.0"
- board text removed: "Sunrise clock display board V1.0, 2021-04-09 https://github.com/atoomnetmarc/Sunrise-clock-hardware Apache License, Version 2.0"

Commit message: Added gerbers and bom.
Other:
- board text added: "Sunrise clock display board V1.0, 2021-04-11 https://github.com/atoomnetmarc/Sunrise-clock-hardware Apache License, Version 2.0"
- board text removed: "Sunrise clock display board V1.0, 2021-04-10 https://github.com/atoomnetmarc/Sunrise-clock-hardware Apache License, Version 2.0"
