File: Sunrise clock display board/Sunrise clock display board.sch (KiCad schematic (older format))
At the start: 20 parts, among them J1 Conn_02x05_Odd_Even, Q1 2N7002, U1 Nokia_5110_display, U2 Nokia_5110_display, U3 Nokia_5110_display

Commit message: Now in stereo if you want.
Parts:
- added LOGO1: Logo_Open_Hardware_Large, Symbol:OSHW-Logo_19x20mm_SilkScreen, symbol Graphic:Logo_Open_Hardware_Large
Changed lines of the file:
@@
 Sheet 1 1
 Title "Sunrise clock display board"
-Date "2021-04-09"
+Date "2021-04-10"
 Rev "V1.0"
 Comp ""
@@
 Wire Wire Line
 	2750 4000 2750 4100
+$Comp
+L Graphic:Logo_Open_Hardware_Large LOGO1
+U 1 1 60719F19
+P 1200 6100
+F 0 "LOGO1" H 1200 6600 50  0001 C CNN
+F 1 "Logo_Open_Hardware_Large" H 1200 5700 50  0001 C CNN
+F 2 "Symbol:OSHW-Logo_19x20mm_SilkScreen" H 1200 6100 50  0001 C CNN
+F 3 "~" H 1200 6100 50  0001 C CNN
+	1    1200 6100
+	1    0    0    -1
+$EndComp
 $EndSCHEMATC
