File: Sunrise clock main board/Sunrise clock main board.kicad_pcb (KiCad board)
At the start: 2 copper layers, 160 x 106.7 mm, 132 parts, among them J1 Barrel_Jack_Switch, J3 Screw terminal/dnf, J4 Conn_02x05_Odd_Even, J5 Conn_01x04_Male, J6 Conn_01x04_Male, Q1 IRML2244, Q2 IRML2244, Q3 2N7002, Q4 2N7002, SW1 SW_Push, SW2 SW_Push, SW3 SW_Push, SW4 SW_Push, SW5 SW_Push, SW6 SW_Push, SW7 SW_Push, SW8 SW_Push, U1 NCP1117LPST33T3G, U10 74HC138D, U2 MAX809S, U3 LM358DR, U4 DS3231MZ, U5 AT24C512C-SSHD, U6 PCA9306DCTR, U7 74AHCT125D, U8 74HC4066D, U9 MCP23017_SP

Commit message: More testing.
Parts:
- added R36: 4k7, Resistor_SMD:R_0805_2012Metric_Pad1.20x1.40mm_HandSolder, F.Cu at (-59.7, 7.62)
- added R47: 10k, Resistor_SMD:R_0805_2012Metric_Pad1.20x1.40mm_HandSolder, F.Cu at (-62.2, 7.62)
Connections:
- A1 pad 6: EXP_INT -> Net-(A1-Pad6)
Routing:
- net Net-(A1-Pad6): track 0.00 -> 5.35 mm
- net EXP_INT: track 55.0 -> 49.9 mm, vias 3 -> 2
Changed lines of the file:
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@@
     (thickness 1.6)
     (drawings 81)
-    (tracks 1521)
+    (tracks 1517)
     (zones 0)
-    (modules 132)
-    (nets 122)
+    (modules 134)
+    (nets 123)
   )
   (page A4)
@@
   (net 120 "Net-(A5-Pad6)")
   (net 121 "Net-(A5-Pad5)")
+  (net 122 "Net-(A1-Pad6)")
   (net_class Default "This is the default net class."
     (clearance 0.2)
@@
     (add_net "Net-(A1-Pad35)")
     (add_net "Net-(A1-Pad37)")
+    (add_net "Net-(A1-Pad6)")
     (add_net "Net-(A3-Pad8)")
     (add_net "Net-(A3-Pad9)")
@@
     (add_net ~SDR)
   )
+  (module Resistor_SMD:R_0805_2012Metric_Pad1.20x1.40mm_HandSolder (layer F.Cu)
+    (at -62.23 7.62 90)
+    (descr "Resistor SMD 0805 (2012 Metric), square (rectangular) end terminal, IPC_7351 nominal with elongated pad for handsoldering. (Body size source: IPC-SM-782 page 72, https://www.pcb-3d.com/wordpress/wp-content/uploads/ipc-sm-782a_amendment_1_and_2.pdf), generated with kicad-footprint-generator")
+    (tags "resistor handsolder")
+    (attr smd)
+    (fp_text reference R47 (at 0 -1.65 90) (layer F.SilkS)
+      (effects (font (size 1 1) (thickness 0.15)))
+    )
+    (fp_text value 10k (at 0 1.65 90) (layer F.Fab)
+      (effects (font (size 1 1) (thickness 0.15)))
+    )
+    (fp_text user %R (at 0 0 90) (layer F.Fab)
+      (effects (font (size 0.5 0.5) (thickness 0.08)))
+    )
+    (fp_line (start -1 0.625) (end -1 -0.625) (layer F.Fab) (width 0.1))
+    (fp_line (start -1 -0.625) (end 1 -0.625) (layer F.Fab) (width 0.1))
+    (fp_line (start 1 -0.625) (end 1 0.625) (layer F.Fab) (width 0.1))
+    (fp_line (start 1 0.625) (end -1 0.625) (layer F.Fab) (width 0.1))
+    (fp_line (start -0.227064 -0.735) (end 0.227064 -0.735) (layer F.SilkS) (width 0.12))
+    (fp_line (start -0.227064 0.735) (end 0.227064 0.735) (layer F.SilkS) (width 0.12))
+    (fp_line (start -1.85 0.95) (end -1.85 -0.95) (layer F.CrtYd) (width 0.05))
+    (fp_line (start -1.85 -0.95) (end 1.85 -0.95) (layer F.CrtYd) (width 0.05))
+    (fp_line (start 1.85 -0.95) (end 1.85 0.95) (layer F.CrtYd) (width 0.05))
+    (fp_line (start 1.85 0.95) (end -1.85 0.95) (layer F.CrtYd) (width 0.05))
+    (pad 2 smd roundrect (at 1 0 90) (size 1.2 1.4) (layers F.Cu F.Paste F.Mask) (roundrect_rratio 0.208333)
+      (net 122 "Net-(A1-Pad6)"))
+    (pad 1 smd roundrect (at -1 0 90) (size 1.2 1.4) (layers F.Cu F.Paste F.Mask) (roundrect_rratio 0.208333)
+      (net 1 GND))
+    (model ${KISYS3DMOD}/Resistor_SMD.3dshapes/R_0805_2012Metric.wrl
+      (at (xyz 0 0 0))
+      (scale (xyz 1 1 1))
+      (rotate (xyz 0 0 0))
+    )
+  )
+  (module Resistor_SMD:R_0805_2012Metric_Pad1.20x1.40mm_HandSolder (layer F.Cu)
+    (at -59.69 7.62 90)
+    (descr "Resistor SMD 0805 (2012 Metric), square (rectangular) end terminal, IPC_7351 nominal with elongated pad for handsoldering. (Body size source: IPC-SM-782 page 72, https://www.pcb-3d.com/wordpress/wp-content/uploads/ipc-sm-782a_amendment_1_and_2.pdf), generated with kicad-footprint-generator")
+    (tags "resistor handsolder")
+    (attr smd)
+    (fp_text reference R36 (at 0 1.905 90) (layer F.SilkS)
+      (effects (font (size 1 1) (thickness 0.15)))
+    )
+    (fp_text value 4k7 (at 0 1.65 90) (layer F.Fab)
+      (effects (font (size 1 1) (thickness 0.15)))
+    )
+    (fp_text user %R (at 0 0 90) (layer F.Fab)
+      (effects (font (size 0.5 0.5) (thickness 0.08)))
+    )
+    (fp_line (start -1 0.625) (end -1 -0.625) (layer F.Fab) (width 0.1))
+    (fp_line (start -1 -0.625) (end 1 -0.625) (layer F.Fab) (width 0.1))
+    (fp_line (start 1 -0.625) (end 1 0.625) (layer F.Fab) (width 0.1))
+    (fp_line (start 1 0.625) (end -1 0.625) (layer F.Fab) (width 0.1))
+    (fp_line (start -0.227064 -0.735) (end 0.227064 -0.735) (layer F.SilkS) (width 0.12))
+    (fp_line (start -0.227064 0.735) (end 0.227064 0.735) (layer F.SilkS) (width 0.12))
+    (fp_line (start -1.85 0.95) (end -1.85 -0.95) (layer F.CrtYd) (width 0.05))
+    (fp_line (start -1.85 -0.95) (end 1.85 -0.95) (layer F.CrtYd) (width 0.05))
+    (fp_line (start 1.85 -0.95) (end 1.85 0.95) (layer F.CrtYd) (width 0.05))
+    (fp_line (start 1.85 0.95) (end -1.85 0.95) (layer F.CrtYd) (width 0.05))
+    (pad 2 smd roundrect (at 1 0 90) (size 1.2 1.4) (layers F.Cu F.Paste F.Mask) (roundrect_rratio 0.208333)
+      (net 122 "Net-(A1-Pad6)"))
+    (pad 1 smd roundrect (at -1 0 90) (size 1.2 1.4) (layers F.Cu F.Paste F.Mask) (roundrect_rratio 0.208333)
+      (net 5 EXP_INT))
+    (model ${KISYS3DMOD}/Resistor_SMD.3dshapes/R_0805_2012Metric.wrl
+      (at (xyz 0 0 0))
+      (scale (xyz 1 1 1))
+      (rotate (xyz 0 0 0))
+    )
+  )
   (module Module-extra:bme280_3V (layer F.Cu)
     (at 47.02 -50.8 90)
@@
       (net 45 "Net-(A1-Pad16)"))
     (pad 6 thru_hole oval (at 0 12.7 90) (size 2.1 1.7) (drill 1) (layers *.Cu *.Mask)
-      (net 5 EXP_INT))
+      (net 122 "Net-(A1-Pad6)"))
     (pad 15 thru_hole oval (at 0 35.56 90) (size 2.1 1.7) (drill 1) (layers *.Cu *.Mask)
       (net 11 SD_SPI_SS))
@@
   (via (at -54.61 33.02) (size 1.6) (drill 0.8) (layers F.Cu B.Cu) (net 1))
   (via (at -59.69 36.83) (size 1.6) (drill 0.8) (layers F.Cu B.Cu) (net 1))
-  (via (at -62.23 7.62) (size 1.6) (drill 0.8) (layers F.Cu B.Cu) (net 1))
   (via (at -30.48 -6.35) (size 1.6) (drill 0.8) (layers F.Cu B.Cu) (net 1))
   (via (at -17.78 -6.35) (size 1.6) (drill 0.8) (layers F.Cu B.Cu) (net 1))
@@
   (via (at -22.86 7.493) (size 0.8) (drill 0.4) (layers F.Cu B.Cu) (net 1))
   (via (at -19.431 8.509) (size 0.8) (drill 0.4) (layers F.Cu B.Cu) (net 1))
+  (via (at -62.23 10.16) (size 0.8) (drill 0.4) (layers F.Cu B.Cu) (net 1))
   (via (at 67.945 -24.638) (size 0.8) (drill 0.4) (layers F.Cu B.Cu) (net 2))
   (segment (start 67.945 -22.895) (end 67.945 -24.638) (width 0.25) (layer F.Cu) (net 2))
@@
   (via (at -43.434 10.287) (size 0.8) (drill 0.4) (layers F.Cu B.Cu) (net 5))
   (segment (start -43.434 10.287) (end -43.434 29.591) (width 0.25) (layer B.Cu) (net 5))
-  (segment (start -59.69 9.144) (end -59.817 9.271) (width 0.25) (layer B.Cu) (net 5))
-  (segment (start -59.69 3.81) (end -59.69 9.144) (width 0.25) (layer B.Cu) (net 5))
-  (via (at -59.817 9.271) (size 0.8) (drill 0.4) (layers F.Cu B.Cu) (net 5))
-  (segment (start -59.436 9.652) (end -59.817 9.271) (width 0.25) (layer F.Cu) (net 5))
-  (segment (start -46.920002 9.652) (end -59.436 9.652) (width 0.25) (layer F.Cu) (net 5))
-  (segment (start -46.006999 9.869001) (end -46.703001 9.869001) (width 0.25) (layer F.Cu) (net 5))
-  (segment (start -45.789998 9.652) (end -46.006999 9.869001) (width 0.25) (layer F.Cu) (net 5))
-  (segment (start -46.703001 9.869001) (end -46.920002 9.652) (width 0.25) (layer F.Cu) (net 5))
-  (segment (start -44.069 9.652) (end -45.789998 9.652) (width 0.25) (layer F.Cu) (net 5))
-  (segment (start -43.434 10.287) (end -44.069 9.652) (width 0.25) (layer F.Cu) (net 5))
   (segment (start -33.614 28.746) (end -33.614 29.871) (width 0.25) (layer F.Cu) (net 5))
   (segment (start -43.034001 29.990999) (end -43.434 29.591) (width 0.25) (layer F.Cu) (net 5))
@@
   (segment (start -34.801965 30.540967) (end -36.701988 32.44099) (width 0.25) (layer F.Cu) (net 5))
   (segment (start -33.614 29.871) (end -34.283967 30.540967) (width 0.25) (layer F.Cu) (net 5))
+  (segment (start -59.69 9.398) (end -59.69 8.62) (width 0.25) (layer F.Cu) (net 5))
+  (segment (start -59.218999 9.869001) (end -59.69 9.398) (width 0.25) (layer F.Cu) (net 5))
+  (segment (start -43.851999 9.869001) (end -59.218999 9.869001) (width 0.25) (layer F.Cu) (net 5))
+  (segment (start -43.434 10.287) (end -43.851999 9.869001) (width 0.25) (layer F.Cu) (net 5))
   (via (at 39.623998 18.922994) (size 0.8) (drill 0.4) (layers F.Cu B.Cu) (net 6))
   (segment (start 53.34 21.59) (end 53.34 25.4) (width 0.25) (layer F.Cu) (net 6))
@@
   (segment (start -20.05 21.352) (end -18.923 22.479) (width 0.25) (layer F.Cu) (net 119))
   (segment (start -20.05 20.32) (end -20.05 21.352) (width 0.25) (layer F.Cu) (net 119))
+  (segment (start -62.23 6.62) (end -59.69 6.62) (width 0.25) (layer F.Cu) (net 122))
+  (segment (start -59.69 6.62) (end -59.69 3.81) (width 0.25) (layer F.Cu) (net 122))
   (zone (net 1) (net_name GND) (layer F.Cu) (hatch edge 0.508)
     (connect_pads (clearance 0.254))

Commit message: More testing.
Parts:
- removed the R13 at (64.5, 3.81)
- removed R20: 1k, Resistor_SMD:R_0805_2012Metric_Pad1.20x1.40mm_HandSolder
- removed R35: 4k7, Resistor_SMD:R_0805_2012Metric_Pad1.20x1.40mm_HandSolder
- removed the R60 at (66.0, -7.62)
- removed TP2, TP5: TestPoint, TestPoint:TestPoint_THTPad_1.5x1.5mm_Drill0.7mm
- added C18: 100nF, Capacitor_SMD:C_0805_2012Metric_Pad1.18x1.45mm_HandSolder, F.Cu at (-14.0, -21.6)
- added NT2: Net-Tie_2, NetTie-fixed:NetTie-2_SMD_Pad0.5mm, F.Cu at (1.41, -38.7)
- added R16: 10R, Resistor_SMD:R_0805_2012Metric_Pad1.20x1.40mm_HandSolder, F.Cu at (2.54, -34.3)
- added R17: 10R, Resistor_SMD:R_0805_2012Metric_Pad1.20x1.40mm_HandSolder, F.Cu at (-2.54, -34.3)
- added U11: INA219AIDCNR, Package_TO_SOT_SMD:SOT-23-8, F.Cu at (-10.2, -21.6)
- C5: value 10uF -> 1uF
- R1: value 0R005 -> 0R05
- moved C5 74.5 mm to (-10.2, -25.4), turned to 180 degrees
- moved NT1 15.9 mm to (-1.27, -38.7)
- moved R1 15.9 mm to (0.00, -38.7)
- moved L1 7.62 mm to (0.00, -25.4)
- moved C10 4.58 mm to (73.7, -20.3), turned to 90 degrees
- moved TP19 4.32 mm to (73.9, -27.9)
- moved D1 0.64 mm to (-15.9, -47.0), turned to 90 degrees
- renumbered R16 to R13, R71 to R60
Connections:
- A1 pad 5: EXTERNAL_CURRENT -> Net-(A1-Pad5)
- C10 pad 2: GND2 -> GND
- C5 pad 2: GND2 -> Net-(C5-Pad2)
- D1 pad 2: GND -> Net-(D1-Pad2)
- F2 pad 1: +5V -> Net-(D1-Pad2)
- J1 pad 1: +5VL -> Net-(J1-Pad1)
- J3 pad 1: EXTERNAL_GND -> GND
- NT1 pad 1: GND -> +5VL
- NT1 pad 2: GND2 -> VIN-
- R1 pad 1: GND -> +5VL
- R1 pad 2: EXTERNAL_GND -> Net-(J1-Pad1)
- R40 pad 2: GND2 -> GND
- R80 pad 2: GND2 -> GND
- U3 pad 4: GND2 -> GND
- U3 pad 5: Net-(C5-Pad1) -> GND
- U3 pad 6: Net-(R20-Pad2) -> Net-(U3-Pad6)
- U3 pad 7: Net-(R13-Pad2) -> Net-(U3-Pad6)
Routing:
- net EXTERNAL_CURRENT: track 144.4 -> 0.00 mm, vias 3 -> 0
- net GND2: track 130.5 -> 0.00 mm, vias 4 -> 0
- net EXTERNAL_GND: track 80.0 -> 0.00 mm, vias 2 -> 0
- net Net-(R13-Pad2): track 26.6 -> 0.00 mm, vias 2 -> 0
- net Net-(C5-Pad2): track 0.00 -> 19.9 mm, vias 0 -> 2
- net Net-(R20-Pad2): track 15.1 -> 0.00 mm
- net Net-(J1-Pad1): track 0.00 -> 13.0 mm
- net +3V3: track 433.9 -> 444.1 mm
- net +5V: track 429.3 -> 423.3 mm
- net Net-(D1-Pad2): track 0.00 -> 5.81 mm
- net 3V_MCU: track 181.4 -> 175.8 mm
- net Net-(F1-Pad2): track 7.62 -> 13.1 mm
- net SCL_3V: track 238.4 -> 243.6 mm, vias 3 -> 5
- net SDA_3V: track 239.0 -> 244.0 mm, vias 5 -> 7
- net VIN-: track 0.00 -> 4.76 mm
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Other:
- board text added: "Sunrise clock V1.1, 2021-05-04 https://github.com/atoomnetmarc/Sunrise-clock-hardware Apache License, Version 2.0"
- board text removed: "Sunrise clock V1.1, 2021-05-03 https://github.com/atoomnetmarc/Sunrise-clock-hardware Apache License, Version 2.0"
- board text removed: "Vshunt"
- board text removed: "Vshunt*gain"
