File: Sunrise clock main board/Control.sch (KiCad schematic (older format))
At the start: 29 parts, among them J5 Conn_01x04_Male, J6 Conn_01x04_Male, J7 Conn_01x05_Male, U10 74HC138D, U6 PCA9306DCTR, U9 MCP23017_SP

Commit message: Tweaks
Parts:
- renumbered C27 to C14
Changed lines of the file:
@@
 P 2100 6500
 AR Path="/6087DFFC" Ref="C?"  Part="1"
-AR Path="/6000DF4A/6087DFFC" Ref="C27"  Part="1"
-F 0 "C27" H 2215 6546 50  0000 L CNN
+AR Path="/6000DF4A/6087DFFC" Ref="C14"  Part="1"
+F 0 "C14" H 2215 6546 50  0000 L CNN
 F 1 "100nF" H 2215 6455 50  0000 L CNN
 F 2 "Capacitor_SMD:C_0805_2012Metric_Pad1.18x1.45mm_HandSolder" H 2138 6350 50  0001 C CNN

Commit message: Now in stereo if you want.
Parts:
- removed F5: Polyfuse 250mA >=6V, Fuse:Fuse_1206_3216Metric_Pad1.42x1.75mm_HandSolder, symbol Device:Polyfuse
- removed J7: Conn_01x05_Male, Connector_PinHeader_2.54mm:PinHeader_1x05_P2.54mm_Vertical, symbol Connector:Conn_01x05_Male
- removed R62: 100k, Resistor_SMD:R_0805_2012Metric_Pad1.20x1.40mm_HandSolder, symbol Device:R
- added R71: 100k, Resistor_SMD:R_0805_2012Metric_Pad1.20x1.40mm_HandSolder, symbol Device:R
- added TP18: TestPoint, TestPoint:TestPoint_THTPad_1.5x1.5mm_Drill0.7mm, symbol Connector:TestPoint
- renumbered R51 to R78
Connections:
- net labels added: EXTERNAL_CURRENT, GPIO1, GPIO33, GPIO5, GPO2, I2S_GAIN0, I2S_GAIN1
- net labels removed: GPB0, GPB1, GPB2, I2S_GAIN, IO33, IO5, NEOPIXEL_POWER
- wire segments 149 -> 143
Other:
- moved on the sheet: C14, R5, R6, R61, R7, R8, U10

Commit message: Start of V1.1
Parts:
- removed C18: 100nF, Capacitor_SMD:C_0805_2012Metric_Pad1.18x1.45mm_HandSolder, symbol Device:C
Connections:
- net +5V: no longer U6.7 (VREF2)
- net at C1.1, R78.2, U6.8 (EN): now also U6.7 (VREF2)
Changed lines of the file:
@@
 Sheet 6 6
 Title "Sunrise clock main board"
-Date "2021-04-11"
-Rev "V1.0"
+Date "2021-05-02"
+Rev "V1.1"
 Comp "https://github.com/atoomnetmarc/Sunrise-clock-hardware"
 Comment1 ""
@@
 $Comp
 L power:+5V #PWR?
-U 1 1 60027F1E
-P 8400 1100
-AR Path="/60027F1E" Ref="#PWR?"  Part="1"
-AR Path="/6000DF4A/60027F1E" Ref="#PWR0180"  Part="1"
-F 0 "#PWR0180" H 8400 950 50  0001 C CNN
-F 1 "+5V" H 8415 1273 50  0000 C CNN
-F 2 "" H 8400 1100 50  0001 C CNN
-F 3 "" H 8400 1100 50  0001 C CNN
-	1    8400 1100
-	1    0    0    -1
-$EndComp
-Wire Wire Line
-	8400 1450 8400 1100
-$Comp
-L power:+5V #PWR?
 U 1 1 60027F2B
 P 9300 1100
@@
 	9300 2100 9300 1850
 Wire Wire Line
-	8700 1850 9300 1850
+	8700 1850 8800 1850
 Connection ~ 9300 1850
 Text GLabel 9100 4500 2    50   Output ~ 0
@@
 $EndComp
 $Comp
-L Device:C C?
-U 1 1 5FF21F5F
-P 8800 1550
-AR Path="/5FF21F5F" Ref="C?"  Part="1"
-AR Path="/6000DF4A/5FF21F5F" Ref="C18"  Part="1"
-F 0 "C18" H 8915 1596 50  0000 L CNN
-F 1 "100nF" H 8915 1505 50  0000 L CNN
-F 2 "Capacitor_SMD:C_0805_2012Metric_Pad1.18x1.45mm_HandSolder" H 8838 1400 50  0001 C CNN
-F 3 "~" H 8800 1550 50  0001 C CNN
-	1    8800 1550
-	1    0    0    -1
-$EndComp
-$Comp
 L power:+3.3V #PWR?
 U 1 1 5FF221AB
@@
 $EndComp
 $Comp
-L power:+5V #PWR?
-U 1 1 5FF223CA
-P 8800 1100
-AR Path="/5FF223CA" Ref="#PWR?"  Part="1"
-AR Path="/6000DF4A/5FF223CA" Ref="#PWR0181"  Part="1"
-F 0 "#PWR0181" H 8800 950 50  0001 C CNN
-F 1 "+5V" H 8815 1273 50  0000 C CNN
-F 2 "" H 8800 1100 50  0001 C CNN
-F 3 "" H 8800 1100 50  0001 C CNN
-	1    8800 1100
-	1    0    0    -1
-$EndComp
-$Comp
 L power:GND #PWR?
 U 1 1 5FF22625
@@
 Wire Wire Line
 	7600 1400 7600 1100
-Wire Wire Line
-	8800 1100 8800 1400
-Wire Wire Line
-	8800 1700 8800 2650
 $Comp
 L Device:Polyfuse F?
@@
 Wire Wire Line
 	10500 4700 10700 4700
+Wire Wire Line
+	8400 1450 8400 1250
+Wire Wire Line
+	8400 1250 8800 1250
+Wire Wire Line
+	8800 1250 8800 1850
+Connection ~ 8800 1850
+Wire Wire Line
+	8800 1850 9300 1850
 $EndSCHEMATC

Commit message: More testing.
Parts:
- added R36: 4k7, Resistor_SMD:R_0805_2012Metric_Pad1.20x1.40mm_HandSolder, symbol Device:R
- added R47: 10k, Resistor_SMD:R_0805_2012Metric_Pad1.20x1.40mm_HandSolder, symbol Device:R
Connections:
- net EXP_INT: now also R36.1; no longer A1.6 (IO35)
- net GND: now also R47.1
- new net: A1.6 (IO35), R36.2, R47.2
Changed lines of the file:
@@
 Wire Wire Line
 	3650 3200 4000 3200
-Text GLabel 4000 3300 2    50   Input ~ 0
+Text GLabel 5350 2800 2    50   Input ~ 0
 EXP_INT
-Wire Wire Line
-	3650 3300 4000 3300
 $Comp
 L power:GND #PWR?
@@
 Wire Wire Line
 	8800 1850 9300 1850
+$Comp
+L Device:R R?
+U 1 1 60938F94
+P 5050 3100
+AR Path="/60938F94" Ref="R?"  Part="1"
+AR Path="/6000DF4A/60938F94" Ref="R36"  Part="1"
+F 0 "R36" H 5120 3146 50  0000 L CNN
+F 1 "4k7" H 5120 3055 50  0000 L CNN
+F 2 "Resistor_SMD:R_0805_2012Metric_Pad1.20x1.40mm_HandSolder" V 4980 3100 50  0001 C CNN
+F 3 "~" H 5050 3100 50  0001 C CNN
+	1    5050 3100
+	1    0    0    -1
+$EndComp
+$Comp
+L Device:R R?
+U 1 1 60939612
+P 5050 3550
+AR Path="/60939612" Ref="R?"  Part="1"
+AR Path="/6000DF4A/60939612" Ref="R47"  Part="1"
+F 0 "R47" H 4980 3504 50  0000 R CNN
+F 1 "10k" H 4980 3595 50  0000 R CNN
+F 2 "Resistor_SMD:R_0805_2012Metric_Pad1.20x1.40mm_HandSolder" V 4980 3550 50  0001 C CNN
+F 3 "~" H 5050 3550 50  0001 C CNN
+	1    5050 3550
+	-1   0    0    1
+$EndComp
+$Comp
+L power:GND #PWR?
+U 1 1 60939B35
+P 5050 4400
+AR Path="/60939B35" Ref="#PWR?"  Part="1"
+AR Path="/6000DF4A/60939B35" Ref="#PWR0129"  Part="1"
+F 0 "#PWR0129" H 5050 4150 50  0001 C CNN
+F 1 "GND" H 5055 4227 50  0000 C CNN
+F 2 "" H 5050 4400 50  0001 C CNN
+F 3 "" H 5050 4400 50  0001 C CNN
+	1    5050 4400
+	1    0    0    -1
+$EndComp
+Wire Wire Line
+	5050 4400 5050 3700
+Wire Wire Line
+	5050 3400 5050 3300
+Wire Wire Line
+	5050 2950 5050 2800
+Wire Wire Line
+	5050 2800 5350 2800
+Wire Wire Line
+	3650 3300 5050 3300
+Connection ~ 5050 3300
+Wire Wire Line
+	5050 3300 5050 3250
+$Comp
+L power:PWR_FLAG #FLG0105
+U 1 1 6095E361
+P 8800 1100
+F 0 "#FLG0105" H 8800 1175 50  0001 C CNN
+F 1 "PWR_FLAG" H 8800 1273 50  0000 C CNN
+F 2 "" H 8800 1100 50  0001 C CNN
+F 3 "~" H 8800 1100 50  0001 C CNN
+	1    8800 1100
+	1    0    0    -1
+$EndComp
+Wire Wire Line
+	8800 1100 8800 1250
+Connection ~ 8800 1250
 $EndSCHEMATC

Commit message: More testing.
Parts:
- renumbered R71 to R60
Connections:
- net EXTERNAL_CURRENT: no longer names the net of A1.5 (IO34)
- no-connect marks 16 -> 17
Changed lines of the file:
@@
 Sheet 6 6
 Title "Sunrise clock main board"
-Date "2021-05-02"
+Date "2021-05-04"
 Rev "V1.1"
 Comp "https://github.com/atoomnetmarc/Sunrise-clock-hardware"
@@
 Text GLabel 9100 4400 2    50   Input ~ 0
 RTC_INT
-Wire Wire Line
-	3650 3200 4000 3200
 Text GLabel 5350 2800 2    50   Input ~ 0
 EXP_INT
@@
 Wire Wire Line
 	9300 1700 9300 1850
-Text GLabel 4000 3200 2    50   Input ~ 0
-EXTERNAL_CURRENT
 Wire Wire Line
 	8900 4400 9100 4400
@@
 P 10500 4150
 AR Path="/60B7262C" Ref="R?"  Part="1"
-AR Path="/6000DF4A/60B7262C" Ref="R71"  Part="1"
-F 0 "R71" H 10430 4104 50  0000 R CNN
+AR Path="/6000DF4A/60B7262C" Ref="R60"  Part="1"
+F 0 "R60" H 10430 4104 50  0000 R CNN
 F 1 "100k" H 10430 4195 50  0000 R CNN
 F 2 "Resistor_SMD:R_0805_2012Metric_Pad1.20x1.40mm_HandSolder" V 10430 4150 50  0001 C CNN
@@
 	8800 1100 8800 1250
 Connection ~ 8800 1250
+NoConn ~ 3650 3200
 $EndSCHEMATC
