File: Sunrise clock main board/Input.sch (KiCad schematic (older format))
At the start: 42 parts, among them SW1 SW_Push, SW2 SW_Push, SW3 SW_Push, SW4 SW_Push, SW5 SW_Push, SW6 SW_Push, SW7 SW_Push, SW8 SW_Push, U4 DS3231MZ

Commit message: Now in stereo if you want.
Parts:
- removed C19, C20, C21, C22, C23, C24, C25, C26: 100nF, Capacitor_SMD:C_0805_2012Metric_Pad1.18x1.45mm_HandSolder, symbol Device:C
- removed R21, R22, R23, R24, R25, R26, R27, R28: 1k, Resistor_SMD:R_0805_2012Metric_Pad1.20x1.40mm_HandSolder, symbol Device:R
- removed R52, R53, R54, R55, R56, R57, R58, R59: 100k, Resistor_SMD:R_0805_2012Metric_Pad1.20x1.40mm_HandSolder, symbol Device:R
- added TP19: TestPoint, TestPoint:TestPoint_THTPad_1.5x1.5mm_Drill0.7mm, symbol Connector:TestPoint
- renumbered A7 to A5, R47 to R41, R80 to R90
Connections:
- net GND: now also TP19.1
- net GPA0: now also SW1.1
- net GPA1: now also SW2.1
- net GPA2: now also SW3.1
- net GPA3: now also SW4.1
- net GPA4: now also SW5.1
- net GPA5: now also SW6.1
- net GPA6: now also SW7.1
- net GPA7: now also SW8.1
Other:
- moved on the sheet: SW2, SW3, SW4, SW5, SW6, SW7, SW8

Commit message: changed BME280 module to a 3v one
Parts:
- A5: value BME280 module -> BME280 module 3V; footprint Module-extra:bme280 -> Module-extra:bme280_3V; symbol Module-extra:BME280 -> Module-extra:BME280_3V
Connections:
- net +5V is gone; now on net +3V3: A5.1 (VIN)
- no-connect marks 1 -> 3
Changed lines of the file:
@@
 Sheet 4 6
 Title "Sunrise clock main board"
-Date "2021-04-11"
+Date "2021-05-03"
 Rev "V1.0"
 Comp "https://github.com/atoomnetmarc/Sunrise-clock-hardware"
@@
 I2C: 0x68
 $Comp
-L Module-extra:BME280 U?
+L Module-extra:BME280_3V U?
 U 1 1 5FEE6C4C
 P 1950 7150
@@
 AR Path="/5FE8F2D8/5FEE6C4C" Ref="A5"  Part="1"
 F 0 "A5" H 2228 7346 50  0000 L CNN
-F 1 "BME280 module" H 2228 7255 50  0000 L CNN
-F 2 "Module-extra:bme280" H 1950 7150 50  0001 C CNN
+F 1 "BME280 module 3V" H 2228 7255 50  0000 L CNN
+F 2 "Module-extra:bme280_3V" H 1950 7150 50  0001 C CNN
 F 3 "" H 1950 7150 50  0001 C CNN
 	1    1950 7150
@@
 $EndComp
 Wire Wire Line
-	1350 7050 1600 7050
-Wire Wire Line
-	1600 6950 1350 6950
-Text GLabel 1350 6950 0    50   Input ~ 0
+	1350 6950 1600 6950
+Wire Wire Line
+	1600 6850 1350 6850
+Text GLabel 1350 6850 0    50   Input ~ 0
 SCL_3V
-Text GLabel 1350 7050 0    50   BiDi ~ 0
+Text GLabel 1350 6950 0    50   BiDi ~ 0
 SDA_3V
 $Comp
@@
 Text Notes 2250 7200 0    50   ~ 0
 I2C: 0x76
-$Comp
-L power:+5V #PWR0153
-U 1 1 60122BD7
-P 1950 6550
-F 0 "#PWR0153" H 1950 6400 50  0001 C CNN
-F 1 "+5V" H 1965 6723 50  0000 C CNN
-F 2 "" H 1950 6550 50  0001 C CNN
-F 3 "" H 1950 6550 50  0001 C CNN
-	1    1950 6550
-	1    0    0    -1
-$EndComp
 $Comp
 L Connector:TestPoint TP?
@@
 Wire Wire Line
 	3550 5000 3550 4800
+NoConn ~ 1600 7050
+NoConn ~ 1600 7150
+$Comp
+L power:+3.3V #PWR?
+U 1 1 609048B1
+P 1950 6550
+AR Path="/609048B1" Ref="#PWR?"  Part="1"
+AR Path="/5FE8F2D8/609048B1" Ref="#PWR?"  Part="1"
+F 0 "#PWR?" H 1950 6400 50  0001 C CNN
+F 1 "+3.3V" H 1965 6723 50  0000 C CNN
+F 2 "" H 1950 6550 50  0001 C CNN
+F 3 "" H 1950 6550 50  0001 C CNN
+	1    1950 6550
+	1    0    0    -1
+$EndComp
 $EndSCHEMATC
