File: Sunrise clock main board/Storage.sch (KiCad schematic (older format))
At the start: 17 parts, among them U5 AT24C32N, U8 74HC4066D

Commit message: Tweaks
Parts:
- U5: value AT24C32N -> AT24C512C-SSHD
- renumbered C14 to C6
Changed lines of the file:
@@
 P 10050 2100
 AR Path="/6000A5BE" Ref="C?"  Part="1"
-AR Path="/5FFF46F4/6000A5BE" Ref="C14"  Part="1"
-F 0 "C14" H 10165 2146 50  0000 L CNN
+AR Path="/5FFF46F4/6000A5BE" Ref="C6"  Part="1"
+F 0 "C6" H 10165 2146 50  0000 L CNN
 F 1 "10uF" H 10165 2055 50  0000 L CNN
 F 2 "Capacitor_SMD:C_0805_2012Metric_Pad1.18x1.45mm_HandSolder" H 10088 1950 50  0001 C CNN
@@
 P 2250 4800
 F 0 "U5" H 2450 5050 50  0000 C CNN
-F 1 "AT24C32N" H 2450 4550 50  0000 C CNN
+F 1 "AT24C512C-SSHD" H 2650 4550 50  0000 C CNN
 F 2 "Package_SO:SOIC-8_3.9x4.9mm_P1.27mm" H 2250 4800 50  0001 C CNN
 F 3 "" H 2250 4800 50  0001 C CNN

Commit message: Now in stereo if you want.
Changed lines of the file:
@@
 Sheet 5 6
 Title "Sunrise clock main board"
-Date "2021-04-09"
+Date "2021-04-10"
 Rev "V1.0"
 Comp ""
@@
 AR Path="/5FE8F2D8/5FE6D821" Ref="TP?"  Part="1"
 AR Path="/5FFF46F4/5FE6D821" Ref="TP12"  Part="1"
-F 0 "TP12" H 4750 1575 50  0000 C CNN
-F 1 "TestPoint" H 4750 1484 50  0000 C CNN
+F 0 "TP12" H 4650 1450 50  0000 L CNN
+F 1 "TestPoint" H 4750 1484 50  0001 C CNN
 F 2 "TestPoint:TestPoint_THTPad_1.5x1.5mm_Drill0.7mm" H 4950 1250 50  0001 C CNN
 F 3 "~" H 4950 1250 50  0001 C CNN
@@
 AR Path="/5FE8F2D8/5FE7018B" Ref="TP?"  Part="1"
 AR Path="/5FFF46F4/5FE7018B" Ref="TP13"  Part="1"
-F 0 "TP13" H 5100 1575 50  0000 C CNN
-F 1 "TestPoint" H 5100 1484 50  0000 C CNN
+F 0 "TP13" H 5000 1450 50  0000 L CNN
+F 1 "TestPoint" H 5100 1484 50  0001 C CNN
 F 2 "TestPoint:TestPoint_THTPad_1.5x1.5mm_Drill0.7mm" H 5300 1250 50  0001 C CNN
 F 3 "~" H 5300 1250 50  0001 C CNN
@@
 AR Path="/5FE8F2D8/5FE71C10" Ref="TP?"  Part="1"
 AR Path="/5FFF46F4/5FE71C10" Ref="TP14"  Part="1"
-F 0 "TP14" H 5450 1575 50  0000 C CNN
-F 1 "TestPoint" H 5450 1484 50  0000 C CNN
+F 0 "TP14" H 5350 1450 50  0000 L CNN
+F 1 "TestPoint" H 5450 1484 50  0001 C CNN
 F 2 "TestPoint:TestPoint_THTPad_1.5x1.5mm_Drill0.7mm" H 5650 1250 50  0001 C CNN
 F 3 "~" H 5650 1250 50  0001 C CNN
@@
 AR Path="/5FE8F2D8/5FE735F8" Ref="TP?"  Part="1"
 AR Path="/5FFF46F4/5FE735F8" Ref="TP15"  Part="1"
-F 0 "TP15" H 5800 1575 50  0000 C CNN
-F 1 "TestPoint" H 5800 1484 50  0000 C CNN
+F 0 "TP15" H 5700 1450 50  0000 L CNN
+F 1 "TestPoint" H 5800 1484 50  0001 C CNN
 F 2 "TestPoint:TestPoint_THTPad_1.5x1.5mm_Drill0.7mm" H 6000 1250 50  0001 C CNN
 F 3 "~" H 6000 1250 50  0001 C CNN
@@
 AR Path="/5FE8F2D8/5FE75233" Ref="TP?"  Part="1"
 AR Path="/5FFF46F4/5FE75233" Ref="TP16"  Part="1"
-F 0 "TP16" H 6150 1575 50  0000 C CNN
-F 1 "TestPoint" H 6150 1484 50  0000 C CNN
+F 0 "TP16" H 6050 1450 50  0000 L CNN
+F 1 "TestPoint" H 6150 1484 50  0001 C CNN
 F 2 "TestPoint:TestPoint_THTPad_1.5x1.5mm_Drill0.7mm" H 6350 1250 50  0001 C CNN
 F 3 "~" H 6350 1250 50  0001 C CNN
@@
 AR Path="/5FE8F2D8/5FF0A99A" Ref="TP?"  Part="1"
 AR Path="/5FFF46F4/5FF0A99A" Ref="TP1"  Part="1"
-F 0 "TP1" H 7650 3175 50  0000 C CNN
-F 1 "TestPoint" H 7650 3084 50  0000 C CNN
+F 0 "TP1" H 7600 3050 50  0000 L CNN
+F 1 "TestPoint" H 7650 3084 50  0001 C CNN
 F 2 "TestPoint:TestPoint_THTPad_1.5x1.5mm_Drill0.7mm" H 7850 2850 50  0001 C CNN
 F 3 "~" H 7850 2850 50  0001 C CNN
