File: Sunrise clock main board/Sunrise clock main board.sch (KiCad schematic (older format))
At the start: 6 parts

Commit message: Now in stereo if you want.
Parts:
- added LOGO1: Logo_Open_Hardware_Large, Symbol:OSHW-Logo_11.4x12mm_SilkScreen, symbol Graphic:Logo_Open_Hardware_Large
Changed lines of the file:
@@
 Sheet 1 6
 Title "Sunrise clock main board"
-Date "2021-04-09"
+Date "2021-04-10"
 Rev "V1.0"
 Comp ""
@@
 	1950 6900 1950 7500
 Connection ~ 1950 6900
+$Comp
+L Graphic:Logo_Open_Hardware_Large LOGO1
+U 1 1 6072DC7D
+P 1200 6050
+F 0 "LOGO1" H 1200 6550 50  0001 C CNN
+F 1 "Logo_Open_Hardware_Large" H 1200 5650 50  0001 C CNN
+F 2 "Symbol:OSHW-Logo_11.4x12mm_SilkScreen" H 1200 6050 50  0001 C CNN
+F 3 "~" H 1200 6050 50  0001 C CNN
+	1    1200 6050
+	1    0    0    -1
+$EndComp
 $EndSCHEMATC
